File: 4_Fabrication/Version_0.2/C_KiCad_430476043716/projet.kicad_pcb (KiCad board)
At the start: 2 copper layers, 98 x 187 mm, 139 parts, among them J1 FT232RL, Q1 BC856B, Q2 BC856B, Q3 BC856B, Q4 BC856B, Q5 BC856B, Q6 BC856B, SW1 Wuerth_4.5x6.5mm, SW10 G77, SW11 G77, SW12 G77, SW13 G77, SW14 G77, SW15 G77, SW16 G77, SW17 G77, SW18 G77, SW19 G77, SW2 Wuerth_4.5x6.5mm, SW20 G77, SW21 G77, SW22 G77, SW23 G77, SW24 G77, SW25 G77, SW26 G77, SW27 G77, SW28 G77, SW29 G77, SW3 G77, SW30 G77, SW31 G77, SW32 G77, SW33 G77, SW34 G77, SW35 G77, SW36 G77, SW37 G77, SW38 SK-12F14, SW4 G77, SW5 G77, SW6 G77, SW7 G77, SW8 G77, SW9 G77, U1 Wavga_TP4056, U2 TPS63001DRCR, U3 ESP32-WROOM-32, U4 PCF8574A

Commit message: Commande PCD 25.08.2020 midi
Parts:
- moved C4 0.77 mm to (114.0, 57.9)
Routing:
- net LCD_E: track 249.7 -> 134.7 mm, vias 4 -> 2
- net GND: track 100.9 -> 88.6 mm, vias 87 -> 88
Other:
- board text added: "Polonaise Inverse V0.6 25.08.2020 Sleny Martinez ETML - Près-Apprentissages 2020-2021"
- board text added: "·"
- board text removed: "Polonaise Inverse V0.5 MAS - Franklin·e Berger"
