File: 4_Fabrication/Version_0.2/C_KiCad_430476043716/projet.sch (KiCad schematic (older format))
At the start: 139 parts, among them J1 FT232RL, Q1 BC856B, Q2 BC856B, Q3 BC856B, Q4 BC856B, Q5 BC856B, Q6 BC856B, SW1 Wuerth_4.5x6.5mm, SW10 G77, SW11 G77, SW12 G77, SW13 G77, SW14 G77, SW15 G77, SW16 G77, SW17 G77, SW18 G77, SW19 G77, SW2 Wuerth_4.5x6.5mm, SW20 G77, SW21 G77, SW22 G77, SW23 G77, SW24 G77, SW25 G77, SW26 G77, SW27 G77, SW28 G77, SW29 G77, SW3 G77, SW30 G77, SW31 G77, SW32 G77, SW33 G77, SW34 G77, SW35 G77, SW36 G77, SW37 G77, SW38 SK-12F14, SW4 G77, SW5 G77, SW6 G77, SW7 G77, SW8 G77, SW9 G77, U1 Wavga_TP4056, U2 TPS63001DRCR, U3 ESP32-WROOM-32, U4 PCF8574A

Commit message: Clavier
Parts:
- gave numbers to parts that had none: 2
Changed lines of the file:
@@
 L projet-rescue:+3V3-power #PWR04
 U 1 1 5F793F3E
-P 6200 2025
-F 0 "#PWR04" H 6200 1875 50  0001 C CNN
-F 1 "+3V3" V 6215 2153 50  0000 L CNN
-F 2 "" H 6200 2025 50  0001 C CNN
-F 3 "" H 6200 2025 50  0001 C CNN
-	1    6200 2025
+P 6275 2025
+F 0 "#PWR04" H 6275 1875 50  0001 C CNN
+F 1 "+3V3" V 6290 2153 50  0000 L CNN
+F 2 "" H 6275 2025 50  0001 C CNN
+F 3 "" H 6275 2025 50  0001 C CNN
+	1    6275 2025
 	0    1    1    0
 $EndComp
 Wire Wire Line
-	6200 2025 6125 2025
+	6275 2025 6125 2025
 Connection ~ 5750 2025
 Wire Wire Line
@@
 Ecran LCD\nBacklight
 $Comp
-L archive:Device_LED D?
+L archive:Device_LED D13
 U 1 1 5F9E8C8B
 P 6125 2325
-F 0 "D?" V 6175 2475 50  0000 R CNN
+F 0 "D13" V 6175 2475 50  0000 R CNN
 F 1 "Rouge SMD" V 6100 2800 50  0000 R CNN
 F 2 "LED_SMD:LED_1206_3216Metric_ReverseMount_Hole1.8x2.4mm" H 6125 2325 50  0001 C CNN
@@
 $EndComp
 $Comp
-L archive:Device_R R?
+L archive:Device_R R37
 U 1 1 5F9E8C93
 P 6125 2675
-F 0 "R?" H 5975 2750 50  0000 L CNN
+F 0 "R37" H 5975 2750 50  0000 L CNN
 F 1 "330[Ω]" H 5800 2675 50  0000 L CNN
 F 2 "Resistor_SMD:R_1206_3216Metric_Pad1.42x1.75mm_HandSolder" V 6055 2675 50  0001 C CNN
@@
 	6125 2025 5750 2025
 $Comp
-L archive:power_GND #PWR?
+L archive:power_GND #PWR0101
 U 1 1 5FBAB8D9
 P 6125 2950
-F 0 "#PWR?" H 6125 2700 50  0001 C CNN
+F 0 "#PWR0101" H 6125 2700 50  0001 C CNN
 F 1 "GND" H 6130 2777 50  0000 C CNN
 F 2 "" H 6125 2950 50  0001 C CNN

Commit message: Commande PCD 25.08.2020 midi
Parts:
- BT1: value Litium 3.4[Ah] -> Litium 18650 3.7[V]
- R35: value 6[Ω] -> 5.6[Ω]
Changed lines of the file:
@@
 P 2450 1725
 F 0 "BT1" H 2568 1821 50  0000 L CNN
-F 1 "Litium 3.4[Ah]" H 2568 1730 50  0000 L CNN
+F 1 "Litium 18650 3.7[V]" H 2568 1730 50  0000 L CNN
 F 2 "Battery:BatteryHolder_Aliexpress_XZT_18650" V 2450 1785 50  0001 C CNN
 F 3 "~" V 2450 1785 50  0001 C CNN
@@
 P 12000 2400
 F 0 "R35" H 12000 2250 50  0000 L CNN
-F 1 "6[Ω]" H 12000 2150 50  0000 L CNN
+F 1 "5.6[Ω]" H 12000 2150 50  0000 L CNN
 F 2 "Resistor_SMD:R_1206_3216Metric_Pad1.42x1.75mm_HandSolder" V 11930 2400 50  0001 C CNN
 F 3 "~" H 12000 2400 50  0001 C CNN
@@
 U 1 1 5F9E8C8B
 P 6125 2325
-F 0 "D13" V 6175 2475 50  0000 R CNN
+F 0 "D13" V 6175 2525 50  0000 R CNN
 F 1 "Rouge SMD" V 6100 2800 50  0000 R CNN
 F 2 "LED_SMD:LED_1206_3216Metric_ReverseMount_Hole1.8x2.4mm" H 6125 2325 50  0001 C CNN
